Commit message: worked on simulation

File: graspberry.urdf (robot description, URDF)
Before this commit: robot thorvald_ii, 46 links, 45 joints
Links:
- link /bat0: geometry collision mesh filename=package://Thorvald_Grape_Urdf/meshes/bat_enc_modules/836586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; visual mesh filename=package://Thorvald_Grape_Urdf/meshes/bat_enc_modules/836586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
- link /bat1: geometry collision mesh filename=package://Thorvald_Grape_Urdf/meshes/bat_enc_modules/836586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; visual mesh filename=package://Thorvald_Grape_Urdf/meshes/bat_enc_modules/836586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
- link /corner0_1: geometry collision box size=0.140 0.116 0.058; visual mesh filename=package://Thorvald_Grape_Urdf/meshes/clamps/DUMMY-T-BRACKET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
- link /corner0_2: geometry collision box size=0.140 0.116 0.058; visual mesh filename=package://Thorvald_Grape_Urdf/meshes/clamps/DUMMY-T-BRACKET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
- link /corner1_1: geometry collision box size=0.140 0.116 0.058; visual mesh filename=package://Thorvald_Grape_Urdf/meshes/clamps/DUMMY-T-BRACKET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
- link /corner1_2: geometry collision box size=0.140 0.116 0.058; visual mesh filename=package://Thorvald_Grape_Urdf/meshes/clamps/DUMMY-T-BRACKET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
- link /corner2_1: geometry collision box size=0.140 0.116 0.058; visual mesh filename=package://Thorvald_Grape_Urdf/meshes/clamps/DUMMY-T-BRACKET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
- link /corner2_2: geometry collision box size=0.140 0.116 0.058; visual mesh filename=package://Thorvald_Grape_Urdf/meshes/clamps/DUMMY-T-BRACKET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
- link /corner3_1: geometry collision box size=0.140 0.116 0.058; visual mesh filename=package://Thorvald_Grape_Urdf/meshes/clamps/DUMMY-T-BRACKET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
- link /corner3_2: geometry collision box size=0.140 0.116 0.058; visual mesh filename=package://Thorvald_Grape_Urdf/meshes/clamps/DUMMY-T-BRACKET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
- link /hokuyo_back: geometry collision box size=0.1 0.1 0.1; visual mesh filename=package://Desktop/Thorvald_Grape_Urdf/meshes/hokuyo/hokuyo.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
- link /hokuyo_front: geometry collision box size=0.1 0.1 0.1; visual mesh filename=package://Desktop/Thorvald_Grape_Urdf/meshes/hokuyo/hokuyo.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
- link /leg0: geometry collision mesh filename=package://Thorvald_Grape_Urdf/meshes/drive_modules/836745-5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; visual mesh filename=package://Thorvald_Grape_Urdf/meshes/drive_modules/836745-5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
- link /leg1: geometry collision mesh filename=package://Thorvald_Grape_Urdf/meshes/drive_modules/836745-5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; visual mesh filename=package://Thorvald_Grape_Urdf/meshes/drive_modules/836745-5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
- link /leg2: geometry collision mesh filename=package://Thorvald_Grape_Urdf/meshes/drive_modules/836745-5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; visual mesh filename=package://Thorvald_Grape_Urdf/meshes/drive_modules/836745-5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
- link /leg3: geometry collision mesh filename=package://Thorvald_Grape_Urdf/meshes/drive_modules/836745-5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; visual mesh filename=package://Thorvald_Grape_Urdf/meshes/drive_modules/836745-5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
- link /top0: geometry collision mesh filename=package://Thorvald_Grape_Urdf/meshes/tower_modules/DUMMY-TO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; visual mesh filename=package://Thorvald_Grape_Urdf/meshes/tower_modules/DUMMY-TO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
- link /top1: geometry collision mesh filename=package://Thorvald_Grape_Urdf/meshes/tower_modules/DUMMY-TO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; visual mesh filename=package://Thorvald_Grape_Urdf/meshes/tower_modules/DUMMY-TO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
- link /top2: geometry collision mesh filename=package://Thorvald_Grape_Urdf/meshes/tower_modules/DUMMY-TO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; visual mesh filename=package://Thorvald_Grape_Urdf/meshes/tower_modules/DUMMY-TO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
- link /top3: geometry collision mesh filename=package://Thorvald_Grape_Urdf/meshes/tower_modules/DUMMY-TO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; visual mesh filename=package://Thorvald_Grape_Urdf/meshes/tower_modules/DUMMY-TO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
- link uvtun_frame: geometry visual mesh filename=package://Desktop/Thorvald_Grape_Urdf/meshes/uv_frame/uv_ar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
